File: kicad/Electronic.kicad_pcb (KiCad board)
At the start: 2 copper layers, 62.5 x 50 mm, 14 parts, among them J1 BAT, J2 SOL, J3 ANM, J4 GIR, J5 SERIAL, Q1 IRLZ44N, U1 WeMos_D1_mini_pro, U2 MCP1700-330

Commit message: v389 : electronic pcb update
Parts:
- moved J2 0.50 mm to (118.6, 61.0)
- moved J3 0.50 mm to (163.0, 98.0)
- moved J4 0.50 mm to (148.0, 98.0)
Routing:
- net /-OUT: track 49.9 -> 50.9 mm
- net Net-(J3-Pin_5): track 32.3 -> 31.2 mm
- net /3.3V: track 101.8 -> 102.4 mm
- net /VIT: track 27.6 -> 27.1 mm
- net /+SOL: track 7.27 -> 6.77 mm

Commit message: v441 : fix resistor values on PCB
Parts:
- R1: value 330 -> 120K
- R3: value 100K -> 120K
Changed lines of the file:
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@@
 			)
 		)
-		(attr through_hole dnp)
+		(attr through_hole)
 		(duplicate_pad_numbers_are_jumpers no)
 		(fp_line
@@
 			)
 		)
-		(attr through_hole dnp)
+		(attr through_hole)
 		(duplicate_pad_numbers_are_jumpers no)
 		(fp_line
@@
 			)
 		)
-		(property "Value" "330"
+		(property "Value" "120K"
 			(at 4.431494 0.059773 90)
 			(layer "F.Fab")
@@
 			)
 		)
-		(attr through_hole dnp)
+		(attr through_hole)
 		(duplicate_pad_numbers_are_jumpers no)
 		(fp_line
@@
 			)
 		)
-		(attr through_hole dnp)
+		(attr through_hole)
 		(duplicate_pad_numbers_are_jumpers no)
 		(fp_line
@@
 			)
 		)
-		(attr through_hole dnp)
+		(attr through_hole)
 		(duplicate_pad_numbers_are_jumpers no)
 		(fp_line
@@
 			)
 		)
-		(attr through_hole dnp)
+		(attr through_hole)
 		(duplicate_pad_numbers_are_jumpers no)
 		(fp_line
@@
 			)
 		)
-		(property "Value" "100K"
+		(property "Value" "120K"
 			(at 10.883405 -0.020104 90)
 			(layer "F.Fab")
@@
 			)
 		)
-		(attr through_hole dnp)
+		(attr through_hole)
 		(duplicate_pad_numbers_are_jumpers no)
 		(fp_line
@@
 			)
 		)
-		(attr through_hole dnp)
+		(attr through_hole)
 		(duplicate_pad_numbers_are_jumpers no)
 		(fp_line
@@
 			)
 		)
-		(attr through_hole dnp)
+		(attr through_hole)
 		(duplicate_pad_numbers_are_jumpers no)
 		(fp_line
@@
 			)
 		)
-		(attr through_hole dnp)
+		(attr through_hole)
 		(duplicate_pad_numbers_are_jumpers no)
 		(fp_line
@@
 			)
 		)
-		(attr through_hole dnp)
+		(attr through_hole)
 		(duplicate_pad_numbers_are_jumpers no)
 		(fp_line
@@
 			)
 		)
-		(attr through_hole dnp)
+		(attr through_hole)
 		(duplicate_pad_numbers_are_jumpers no)
 		(fp_line
@@
 			)
 		)
-		(attr through_hole dnp)
+		(attr through_hole)
 		(duplicate_pad_numbers_are_jumpers no)
 		(fp_line
@@
 			)
 		)
-		(attr through_hole dnp)
+		(attr through_hole)
 		(duplicate_pad_numbers_are_jumpers no)
 		(fp_line
